File: hardware/0.1/keyboard.kicad_pcb (KiCad board)
At the start: 2 copper layers, 387 x 120 mm, 327 parts, among them J1 USB_C_Receptacle_USB2.0, J2 SWD, Q1 BSS138, Q2 BSS138, Q3 DTC123J, SW1 SW_Push, U1 USBLC6-2SC6, U2 AP2112K-3.3, U3 STM32F303RCTx, Y1 8MHz

Commit message: continuing layout
Parts:
- added C22: 100n, Capacitor_SMD:C_0603_1608Metric, B.Cu at (345.9, 113.2)
- moved RN4 101.0 mm to (166.6, 110.6), turned to 90 degrees
- moved C13 99.6 mm to (169.2, 110.6), turned to 90 degrees
- moved C10 81.3 mm to (163.9, 110.6), turned to 90 degrees
- moved RN3 77.4 mm to (148.0, 110.7), turned to 90 degrees
- moved C12 76.8 mm to (150.7, 110.7), turned to 90 degrees
- moved C9 71.5 mm to (145.3, 110.7), turned to 90 degrees
- moved RN2 63.2 mm to (128.8, 110.6), turned to 90 degrees
- moved C11 53.6 mm to (131.4, 110.6), turned to 90 degrees
- moved C8 47.4 mm to (126.2, 110.6), turned to 90 degrees
- moved RN1 39.9 mm to (109.7, 110.5), turned to 90 degrees
- moved C6 37.7 mm to (112.3, 110.5), turned to 90 degrees
- moved C7 37.3 mm to (107.0, 110.5), turned to 90 degrees
- moved R5 20.1 mm to (116.5, 103.4)
- moved R6 20.1 mm to (115.0, 103.4)
- moved D_39 19.6 mm to (134.4, 145.1)
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Connections:
- RN1 pad 1: +3V3 -> /ENC0_B_DB
- RN1 pad 3: /ENC0_B_DB -> +3V3
- RN1 pad 6: /ENC0_B -> /ENC0_A
- RN1 pad 7: /ENC0_A -> /ENC0_B
- RN2 pad 1: +3V3 -> /ENC1_B_DB
- RN2 pad 4: +3V3 -> /ENC1_A_DB
- RN2 pad 5: /ENC1_B -> /ENC1_A
- RN2 pad 6: /ENC2_B -> /ENC1_A
- RN2 pad 7: /ENC3_B -> /ENC1_B
- RN2 pad 8: /ENC1_A -> /ENC1_B
- RN3 pad 1: /ENC1_B_DB -> /ENC2_B_DB
- RN3 pad 2: /ENC1_A_DB -> +3V3
- RN3 pad 4: +3V3 -> /ENC2_A_DB
- RN3 pad 6: /ENC3_A -> /ENC2_A
- RN3 pad 7: /ENC1_A -> /ENC2_B
- RN3 pad 8: /ENC1_B -> /ENC2_B
- RN4 pad 2: /ENC3_A_DB -> +3V3
- RN4 pad 3: /ENC2_B_DB -> +3V3
- RN4 pad 4: /ENC2_A_DB -> /ENC3_A_DB
- RN4 pad 5: /ENC2_A -> /ENC3_A
- RN4 pad 6: /ENC2_B -> /ENC3_A
- RN4 pad 7: /ENC3_A -> /ENC3_B
Routing:
- net +5V: track 40.9 -> 1089.9 mm, vias 0 -> 5
- net /col17: track 0.00 -> 116.2 mm
- net /col9: track 0.00 -> 110.0 mm
- net /col7: track 0.00 -> 110.0 mm
- net /col4: track 0.00 -> 108.7 mm
- net /col15: track 0.00 -> 107.1 mm
- net /col10: track 4.76 -> 110.9 mm
- net /col12: track 0.00 -> 106.1 mm
- net /col14: track 4.76 -> 109.9 mm
- net /col16: track 4.76 -> 109.1 mm
- net /col5: track 0.00 -> 104.1 mm
- net /col18: track 0.00 -> 103.1 mm
- net /col19: track 0.00 -> 95.2 mm
- net /col13: track 0.00 -> 86.1 mm
- net /col6: track 0.00 -> 86.1 mm
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