File: hardware/0.1/keyboard.kicad_pcb (KiCad board)
At the start: 2 copper layers, 387 x 120 mm, 328 parts, among them J1 USB_C_Receptacle_USB2.0, J2 SWD, Q1 BSS138, Q2 BSS138, Q3 DTC123J, SW1 SW_Push, U1 USBLC6-2SC6, U2 AP2112K-3.3, U3 STM32F303RCTx, Y1 8MHz

Commit message: layout ++
Parts:
- added BZ1: Buzzer, Buzzer_Beeper:Buzzer_Murata_PKMCS0909E4000-R1, B.Cu at (286.0, 147.7)
- moved D_103 2.30 mm to (386.9, 190.7)
- moved D_75 0.15 mm to (450.0, 157.7)
Connections:
- U3 pad 20: (no net) -> /BUZZER
Routing:
- net /row5: track 0.00 -> 387.9 mm, vias 0 -> 8
- net /row4: track 0.00 -> 350.4 mm, vias 0 -> 4
- net /row1: track 0.00 -> 334.1 mm, vias 0 -> 2
- net /row0: track 22.4 -> 335.1 mm
- net /row2: track 0.00 -> 270.2 mm, vias 0 -> 2
- net /row3: track 0.00 -> 267.2 mm, vias 0 -> 2
- net +3V3: track 32.4 -> 167.1 mm, vias 0 -> 2
- net /status: track 1.53 -> 72.7 mm, vias 0 -> 2
- net Net-(D_78-Pad2): track 0.00 -> 17.4 mm
- net Net-(D15-Pad2): track 53.5 -> 43.2 mm, vias 0 -> 2
- net Net-(D_63-Pad2): track 0.00 -> 8.14 mm
- net Net-(D_114-Pad2): track 0.00 -> 5.19 mm
- net Net-(D3-Pad2): track 56.5 -> 59.2 mm
- net Net-(D_103-Pad2): track 10.7 -> 8.63 mm
- net Net-(D_68-Pad2): track 9.38 -> 7.61 mm
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
Commit message: unrouted = 0 with no matrix - mcu connections
Parts:
- moved R8 1.05 mm to (169.0, 129.3)
- moved 10u1 1.05 mm to (173.3, 123.8)
- moved C3 1.05 mm to (169.0, 127.8)
- moved D24 1.05 mm to (171.8, 127.7)
- moved Q3 1.05 mm to (170.8, 123.5)
- moved R10 1.05 mm to (173.7, 126.8)
- moved R7 1.05 mm to (175.2, 126.8)
Connections:
- U3 pad 36: /status -> /underglow
- U3 pad 57: /underglow -> /status
Routing:
- net +3V3: track 167.1 -> 364.7 mm, vias 2 -> 16
- net /BUZZER: track 0.00 -> 117.5 mm
- net /col1: track 0.00 -> 107.5 mm
- net /col2: track 2.04 -> 107.7 mm
- net /row3: track 267.2 -> 355.7 mm, vias 2 -> 6
- net /row2: track 270.2 -> 350.4 mm, vias 2 -> 6
- net /col3: track 37.7 -> 114.8 mm
- net Net-(R10-Pad2): track 5.62 -> 74.7 mm, vias 0 -> 2
- net /nRST: track 9.78 -> 65.6 mm, vias 0 -> 2
- net Net-(D10-Pad2): track 0.00 -> 50.8 mm, vias 0 -> 2
- net /underglow: track 1.57 -> 49.8 mm, vias 0 -> 2
- net /status: track 72.7 -> 115.7 mm, vias 2 -> 6
- net Net-(D10-Pad4): track 0.00 -> 39.5 mm
- net /row0: track 335.1 -> 363.9 mm, vias 0 -> 2
- net /row1: track 334.1 -> 360.8 mm, vias 2 -> 4
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
Commit message: layout done
Parts:
- moved C5 2.28 mm to (193.6, 147.5)
- moved C4 2.04 mm to (193.6, 143.2)
- moved Y1 1.70 mm to (190.8, 145.6)
Connections:
- R7 pad 2: (no net) -> /MCU_RST
- U3 pad 10: (no net) -> /col7
- U3 pad 11: (no net) -> /col6
- U3 pad 2: (no net) -> /col10
- U3 pad 21: (no net) -> /col13
- U3 pad 22: (no net) -> /col14
- U3 pad 23: (no net) -> /col15
- U3 pad 24: (no net) -> /col16
- U3 pad 25: (no net) -> /row5
- U3 pad 26: (no net) -> /row4
- U3 pad 27: (no net) -> /row3
- U3 pad 28: (no net) -> /col3
- U3 pad 29: (no net) -> /col2
- U3 pad 3: (no net) -> /col11
- U3 pad 30: (no net) -> /col1
- U3 pad 33: (no net) -> /col0
- U3 pad 34: (no net) -> /ENC0_A_DB
- U3 pad 35: (no net) -> /ENC0_B_DB
- U3 pad 38: (no net) -> /ENC1_A_DB
- U3 pad 39: (no net) -> /ENC1_B_DB
- U3 pad 4: (no net) -> /col12
- U3 pad 40: (no net) -> /ENC2_A_DB
- U3 pad 41: (no net) -> /ENC2_B_DB
- U3 pad 42: (no net) -> /ENC3_B_DB
- U3 pad 43: (no net) -> /ENC3_A_DB
- U3 pad 50: (no net) -> /MCU_RST
- U3 pad 51: (no net) -> /row0
- U3 pad 52: (no net) -> /row1
- U3 pad 53: (no net) -> /row2
- U3 pad 55: (no net) -> /col17
- U3 pad 56: (no net) -> /col18
- U3 pad 58: (no net) -> /col19
- U3 pad 61: (no net) -> /col5
- U3 pad 62: (no net) -> /col4
- U3 pad 8: (no net) -> /col9
- U3 pad 9: (no net) -> /col8
Routing:
- net /col19: track 95.2 -> 402.2 mm, vias 0 -> 1
- net /col18: track 103.1 -> 381.3 mm, vias 0 -> 1
- net /col17: track 116.2 -> 378.8 mm, vias 0 -> 1
- net /col16: track 109.1 -> 344.9 mm, vias 0 -> 1
- net /col15: track 107.1 -> 322.0 mm, vias 0 -> 1
- net /col14: track 109.9 -> 304.7 mm, vias 0 -> 1
- net /col13: track 86.1 -> 262.3 mm, vias 0 -> 1
- net /col12: track 106.1 -> 248.1 mm, vias 0 -> 1
- net /col11: track 86.1 -> 208.2 mm, vias 0 -> 1
- net /col10: track 110.9 -> 214.0 mm, vias 0 -> 1
- net /ENC0_A_DB: track 2.73 -> 93.9 mm, vias 0 -> 2
- net /ENC0_B_DB: track 2.74 -> 91.8 mm, vias 0 -> 2
- net /col9: track 110.0 -> 194.2 mm, vias 0 -> 1
- net /ENC1_A_DB: track 2.63 -> 84.5 mm, vias 0 -> 2
- net /ENC1_B_DB: track 2.77 -> 78.8 mm, vias 0 -> 2
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- added copper zone on B.Cu, net GND
