File: hardware/0.1/keyboard.sch (KiCad schematic (older format))
At the start: 327 parts, among them J1 USB_C_Receptacle_USB2.0, J2 SWD, Q1 BSS138, Q2 BSS138, Q3 DTC123J, SW1 SW_Push, U1 USBLC6-2SC6, U2 AP2112K-3.3, U3 STM32F303RCTx, Y1 8MHz

Commit message: continuing layout
Parts:
- added C22: 100n, Capacitor_SMD:C_0603_1608Metric, symbol Device:C
Connections:
- wire segments 829 -> 831
Changed lines of the file:
@@
 $Comp
 L josh-passive:RN RN1
-U 2 1 6AD4FA57
+U 4 1 6AD4FA57
 P 11900 9300
 F 0 "RN1" H 11900 9200 50  0000 C CNN
@@
 F 2 "Resistor_SMD:R_Array_Convex_4x0603" V 11900 9300 50  0001 C CNN
 F 3 "~" V 11900 9300 50  0001 C CNN
-	2    11900 9300
+	4    11900 9300
 	-1   0    0    -1
 $EndComp
 $Comp
 L josh-passive:RN RN1
-U 4 1 6ADCC12F
+U 3 1 6ADCC12F
 P 11250 9000
 F 0 "RN1" V 11204 9068 50  0000 L CNN
@@
 F 2 "Resistor_SMD:R_Array_Convex_4x0603" V 11250 9000 50  0001 C CNN
 F 3 "~" V 11250 9000 50  0001 C CNN
-	4    11250 9000
+	3    11250 9000
 	0    -1   1    0
 $EndComp
 $Comp
 L josh-passive:RN RN1
-U 3 1 6ADCC9F2
+U 2 1 6ADCC9F2
 P 11600 9000
 F 0 "RN1" V 11554 9068 50  0000 L CNN
@@
 F 2 "Resistor_SMD:R_Array_Convex_4x0603" V 11600 9000 50  0001 C CNN
 F 3 "~" V 11600 9000 50  0001 C CNN
-	3    11600 9000
+	2    11600 9000
 	0    -1   1    0
 $EndComp
@@
 Text Label 10800 9300 0    50   ~ 0
 ENC0_B
-$Comp
-L josh-passive:RN RN3
-U 3 1 6B8D177C
-P 11900 10200
-F 0 "RN3" H 11900 10300 50  0000 C CNN
-F 1 "10K" H 11900 10200 50  0000 C CNN
-F 2 "Resistor_SMD:R_Array_Convex_4x0603" V 11900 10200 50  0001 C CNN
-F 3 "~" V 11900 10200 50  0001 C CNN
-	3    11900 10200
-	-1   0    0    -1
-$EndComp
-$Comp
-L josh-passive:RN RN3
-U 4 1 6B8D1782
-P 11900 10300
-F 0 "RN3" H 11900 10200 50  0000 C CNN
-F 1 "10K" H 11900 10300 50  0000 C CNN
-F 2 "Resistor_SMD:R_Array_Convex_4x0603" V 11900 10300 50  0001 C CNN
-F 3 "~" V 11900 10300 50  0001 C CNN
-	4    11900 10300
-	-1   0    0    -1
-$EndComp
-$Comp
-L josh-passive:RN RN2
-U 1 1 6B8D1788
-P 11250 10000
-F 0 "RN2" V 11204 10068 50  0000 L CNN
-F 1 "10K" V 11295 10068 50  0000 L CNN
-F 2 "Resistor_SMD:R_Array_Convex_4x0603" V 11250 10000 50  0001 C CNN
-F 3 "~" V 11250 10000 50  0001 C CNN
-	1    11250 10000
-	0    -1   1    0
-$EndComp
-$Comp
-L josh-passive:RN RN2
-U 4 1 6B8D178E
-P 11600 10000
-F 0 "RN2" V 11554 10068 50  0000 L CNN
-F 1 "10K" V 11645 10068 50  0000 L CNN
-F 2 "Resistor_SMD:R_Array_Convex_4x0603" V 11600 10000 50  0001 C CNN
-F 3 "~" V 11600 10000 50  0001 C CNN
-	4    11600 10000
-	0    -1   1    0
-$EndComp
 Wire Wire Line
 	11750 10200 11600 10200
@@
 Text Label 10800 10300 0    50   ~ 0
 ENC1_B
-$Comp
-L josh-passive:RN RN4
-U 1 1 6B958D98
-P 11900 11150
-F 0 "RN4" H 11900 11250 50  0000 C CNN
-F 1 "10K" H 11900 11150 50  0000 C CNN
-F 2 "Resistor_SMD:R_Array_Convex_4x0603" V 11900 11150 50  0001 C CNN
-F 3 "~" V 11900 11150 50  0001 C CNN
-	1    11900 11150
-	-1   0    0    -1
-$EndComp
-$Comp
-L josh-passive:RN RN4
-U 2 1 6B958D9E
-P 11900 11250
-F 0 "RN4" H 11900 11150 50  0000 C CNN
-F 1 "10K" H 11900 11250 50  0000 C CNN
-F 2 "Resistor_SMD:R_Array_Convex_4x0603" V 11900 11250 50  0001 C CNN
-F 3 "~" V 11900 11250 50  0001 C CNN
-	2    11900 11250
-	-1   0    0    -1
-$EndComp
-$Comp
-L josh-passive:RN RN2
-U 2 1 6B958DA4
-P 11250 10950
-F 0 "RN2" V 11204 11018 50  0000 L CNN
-F 1 "10K" V 11295 11018 50  0000 L CNN
-F 2 "Resistor_SMD:R_Array_Convex_4x0603" V 11250 10950 50  0001 C CNN
-F 3 "~" V 11250 10950 50  0001 C CNN
-	2    11250 10950
-	0    -1   1    0
-$EndComp
-$Comp
-L josh-passive:RN RN3
-U 1 1 6B958DAA
-P 11600 10950
-F 0 "RN3" V 11554 11018 50  0000 L CNN
-F 1 "10K" V 11645 11018 50  0000 L CNN
-F 2 "Resistor_SMD:R_Array_Convex_4x0603" V 11600 10950 50  0001 C CNN
-F 3 "~" V 11600 10950 50  0001 C CNN
-	1    11600 10950
-	0    -1   1    0
-$EndComp
 Wire Wire Line
 	11750 11150 11600 11150
@@
 Text Label 10800 11250 0    50   ~ 0
 ENC2_B
-$Comp
-L josh-passive:RN RN4
-U 3 1 6B9E5982
-P 11900 12050
-F 0 "RN4" H 11900 12150 50  0000 C CNN
-F 1 "10K" H 11900 12050 50  0000 C CNN
-F 2 "Resistor_SMD:R_Array_Convex_4x0603" V 11900 12050 50  0001 C CNN
-F 3 "~" V 11900 12050 50  0001 C CNN
-	3    11900 12050
-	-1   0    0    -1
-$EndComp
-$Comp
-L josh-passive:RN RN4
-U 4 1 6B9E5988
-P 11900 12150
-F 0 "RN4" H 11900 12050 50  0000 C CNN
-F 1 "10K" H 11900 12150 50  0000 C CNN
-F 2 "Resistor_SMD:R_Array_Convex_4x0603" V 11900 12150 50  0001 C CNN
-F 3 "~" V 11900 12150 50  0001 C CNN
-	4    11900 12150
-	-1   0    0    -1
-$EndComp
-$Comp
-L josh-passive:RN RN2
-U 3 1 6B9E598E
-P 11250 11850
-F 0 "RN2" V 11204 11918 50  0000 L CNN
-F 1 "10K" V 11295 11918 50  0000 L CNN
-F 2 "Resistor_SMD:R_Array_Convex_4x0603" V 11250 11850 50  0001 C CNN
-F 3 "~" V 11250 11850 50  0001 C CNN
-	3    11250 11850
-	0    -1   1    0
-$EndComp
-$Comp
-L josh-passive:RN RN3
-U 2 1 6B9E5994
-P 11600 11850
-F 0 "RN3" V 11554 11918 50  0000 L CNN
-F 1 "10K" V 11645 11918 50  0000 L CNN
-F 2 "Resistor_SMD:R_Array_Convex_4x0603" V 11600 11850 50  0001 C CNN
-F 3 "~" V 11600 11850 50  0001 C CNN
-	2    11600 11850
-	0    -1   1    0
-$EndComp
 Wire Wire Line
 	11750 12050 11600 12050
@@
 Wire Wire Line
 	11250 15300 11350 15300
+$Comp
+L josh-passive:RN RN2
+U 2 1 5F31F943
+P 11600 10000
+F 0 "RN2" V 11554 10068 50  0000 L CNN
+F 1 "10K" V 11645 10068 50  0000 L CNN
+F 2 "Resistor_SMD:R_Array_Convex_4x0603" V 11600 10000 50  0001 C CNN
+F 3 "~" V 11600 10000 50  0001 C CNN
+	2    11600 10000
+	0    -1   1    0
+$EndComp
+$Comp
+L josh-passive:RN RN2
+U 4 1 5F31F937
+P 11900 10300
+F 0 "RN2" H 11900 10200 50  0000 C CNN
+F 1 "10K" H 11900 10300 50  0000 C CNN
+F 2 "Resistor_SMD:R_Array_Convex_4x0603" V 11900 10300 50  0001 C CNN
+F 3 "~" V 11900 10300 50  0001 C CNN
+	4    11900 10300
+	-1   0    0    -1
+$EndComp
+$Comp
+L josh-passive:RN RN2
+U 1 1 5F31F931
+P 11900 10200
+F 0 "RN2" H 11900 10300 50  0000 C CNN
+F 1 "10K" H 11900 10200 50  0000 C CNN
+F 2 "Resistor_SMD:R_Array_Convex_4x0603" V 11900 10200 50  0001 C CNN
+F 3 "~" V 11900 10200 50  0001 C CNN
+	1    11900 10200
+	-1   0    0    -1
+$EndComp
+$Comp
+L josh-passive:RN RN2
+U 3 1 5F31F93D
+P 11250 10000
+F 0 "RN2" V 11204 10068 50  0000 L CNN
+F 1 "10K" V 11295 10068 50  0000 L CNN
+F 2 "Resistor_SMD:R_Array_Convex_4x0603" V 11250 10000 50  0001 C CNN
+F 3 "~" V 11250 10000 50  0001 C CNN
+	3    11250 10000
+	0    -1   1    0
+$EndComp
+$Comp
+L josh-passive:RN RN3
+U 2 1 6008D0F2
+P 11600 10950
+F 0 "RN3" V 11554 11018 50  0000 L CNN
+F 1 "10K" V 11645 11018 50  0000 L CNN
+F 2 "Resistor_SMD:R_Array_Convex_4x0603" V 11600 10950 50  0001 C CNN
+F 3 "~" V 11600 10950 50  0001 C CNN
+	2    11600 10950
+	0    -1   1    0
+$EndComp
+$Comp
+L josh-passive:RN RN3
+U 4 1 6008D0F8
+P 11900 11250
+F 0 "RN3" H 11900 11150 50  0000 C CNN
+F 1 "10K" H 11900 11250 50  0000 C CNN
+F 2 "Resistor_SMD:R_Array_Convex_4x0603" V 11900 11250 50  0001 C CNN
+F 3 "~" V 11900 11250 50  0001 C CNN
+	4    11900 11250
+	-1   0    0    -1
+$EndComp
+$Comp
+L josh-passive:RN RN3
+U 1 1 6008D0FE
+P 11900 11150
+F 0 "RN3" H 11900 11250 50  0000 C CNN
+F 1 "10K" H 11900 11150 50  0000 C CNN
+F 2 "Resistor_SMD:R_Array_Convex_4x0603" V 11900 11150 50  0001 C CNN
+F 3 "~" V 11900 11150 50  0001 C CNN
+	1    11900 11150
+	-1   0    0    -1
+$EndComp
+$Comp
+L josh-passive:RN RN3
+U 3 1 6008D104
+P 11250 10950
+F 0 "RN3" V 11204 11018 50  0000 L CNN
+F 1 "10K" V 11295 11018 50  0000 L CNN
+F 2 "Resistor_SMD:R_Array_Convex_4x0603" V 11250 10950 50  0001 C CNN
+F 3 "~" V 11250 10950 50  0001 C CNN
+	3    11250 10950
+	0    -1   1    0
+$EndComp
+$Comp
+L josh-passive:RN RN4
+U 2 1 6014925B
+P 11600 11850
+F 0 "RN4" V 11554 11918 50  0000 L CNN
+F 1 "10K" V 11645 11918 50  0000 L CNN
+F 2 "Resistor_SMD:R_Array_Convex_4x0603" V 11600 11850 50  0001 C CNN
+F 3 "~" V 11600 11850 50  0001 C CNN
+	2    11600 11850
+	0    -1   1    0
+$EndComp
+$Comp
+L josh-passive:RN RN4
+U 3 1 60149261
+P 11250 11850
+F 0 "RN4" V 11204 11918 50  0000 L CNN
+F 1 "10K" V 11295 11918 50  0000 L CNN
+F 2 "Resistor_SMD:R_Array_Convex_4x0603" V 11250 11850 50  0001 C CNN
+F 3 "~" V 11250 11850 50  0001 C CNN
+	3    11250 11850
+	0    -1   1    0
+$EndComp
+$Comp
+L josh-passive:RN RN4
+U 4 1 601FBB3C
+P 11900 12150
+F 0 "RN4" H 11900 12050 50  0000 C CNN
+F 1 "10K" H 11900 12150 50  0000 C CNN
+F 2 "Resistor_SMD:R_Array_Convex_4x0603" V 11900 12150 50  0001 C CNN
+F 3 "~" V 11900 12150 50  0001 C CNN
+	4    11900 12150
+	-1   0    0    -1
+$EndComp
+$Comp
+L josh-passive:RN RN4
+U 1 1 601FBB42
+P 11900 12050
+F 0 "RN4" H 11900 12150 50  0000 C CNN
+F 1 "10K" H 11900 12050 50  0000 C CNN
+F 2 "Resistor_SMD:R_Array_Convex_4x0603" V 11900 12050 50  0001 C CNN
+F 3 "~" V 11900 12050 50  0001 C CNN
+	1    11900 12050
+	-1   0    0    -1
+$EndComp
+$Comp
+L Device:C C?
+U 1 1 602E4E7C
+P 9700 14550
+AR Path="/618A4248/602E4E7C" Ref="C?"  Part="1"
+AR Path="/602E4E7C" Ref="C22"  Part="1"
+F 0 "C22" H 9585 14504 50  0000 R CNN
+F 1 "100n" H 9585 14595 50  0000 R CNN
+F 2 "Capacitor_SMD:C_0603_1608Metric" H 9738 14400 50  0001 C CNN
+F 3 "~" H 9700 14550 50  0001 C CNN
+F 4 "C15849" H 9700 14550 50  0001 C CNN "LCSC"
+F 5 "CL10A105MP8NNNC " H 9700 14550 50  0001 C CNN "MPN"
+F 6 "1276-1866-1-ND " H 9700 14550 50  0001 C CNN "DigiKey"
+F 7 "Samsung Electro-Mechanics" H 9700 14550 50  0001 C CNN "Manufacturer"
+	1    9700 14550
+	-1   0    0    1
+$EndComp
+Wire Wire Line
+	9700 14750 9700 14700
+$Comp
+L power:GND #PWR?
+U 1 1 602E4E83
+P 9700 14750
+AR Path="/618A4248/602E4E83" Ref="#PWR?"  Part="1"
+AR Path="/602E4E83" Ref="#PWR0143"  Part="1"
+F 0 "#PWR0143" H 9700 14500 50  0001 C CNN
+F 1 "GND" H 9705 14577 50  0000 C CNN
+F 2 "" H 9700 14750 50  0001 C CNN
+F 3 "" H 9700 14750 50  0001 C CNN
+	1    9700 14750
+	1    0    0    -1
+$EndComp
+Wire Wire Line
+	9700 14400 9700 14350
+$Comp
+L power:+5V #PWR0156
+U 1 1 602E4E8A
+P 9700 14350
+F 0 "#PWR0156" H 9700 14200 50  0001 C CNN
+F 1 "+5V" H 9715 14523 50  0000 C CNN
+F 2 "" H 9700 14350 50  0001 C CNN
+F 3 "" H 9700 14350 50  0001 C CNN
+	1    9700 14350
+	1    0    0    -1
+$EndComp
 $EndSCHEMATC
