File: hardware/lower-plate/keyboard.sch (KiCad schematic (older format))
At the start: 13 parts

Commit message: mechanical changes
Parts:
- H1, H10, H11, H12, H2, H3, H4, H5, H6, H7, H8, H9: footprint MountingHole:MountingHole_2.7mm -> MountingHole:MountingHole_2.2mm_M2
Changed lines of the file:
@@
 F 0 "H1" H 14050 14446 50  0000 L CNN
 F 1 "M2.5" H 14050 14355 50  0000 L CNN
-F 2 "MountingHole:MountingHole_2.7mm" H 13950 14400 50  0001 C CNN
+F 2 "MountingHole:MountingHole_2.2mm_M2" H 13950 14400 50  0001 C CNN
 F 3 "~" H 13950 14400 50  0001 C CNN
 F 4 "DNP" H 13950 14400 50  0001 C CNN "DNP"
@@
 F 0 "H2" H 14050 14646 50  0000 L CNN
 F 1 "M2.5" H 14050 14555 50  0000 L CNN
-F 2 "MountingHole:MountingHole_2.7mm" H 13950 14600 50  0001 C CNN
+F 2 "MountingHole:MountingHole_2.2mm_M2" H 13950 14600 50  0001 C CNN
 F 3 "~" H 13950 14600 50  0001 C CNN
 F 4 "DNP" H 13950 14600 50  0001 C CNN "DNP"
@@
 F 0 "H3" H 14050 14846 50  0000 L CNN
 F 1 "M2.5" H 14050 14755 50  0000 L CNN
-F 2 "MountingHole:MountingHole_2.7mm" H 13950 14800 50  0001 C CNN
+F 2 "MountingHole:MountingHole_2.2mm_M2" H 13950 14800 50  0001 C CNN
 F 3 "~" H 13950 14800 50  0001 C CNN
 F 4 "DNP" H 13950 14800 50  0001 C CNN "DNP"
@@
 F 0 "H4" H 14050 15046 50  0000 L CNN
 F 1 "M2.5" H 14050 14955 50  0000 L CNN
-F 2 "MountingHole:MountingHole_2.7mm" H 13950 15000 50  0001 C CNN
+F 2 "MountingHole:MountingHole_2.2mm_M2" H 13950 15000 50  0001 C CNN
 F 3 "~" H 13950 15000 50  0001 C CNN
 F 4 "DNP" H 13950 15000 50  0001 C CNN "DNP"
@@
 F 0 "H5" H 14050 15246 50  0000 L CNN
 F 1 "M2.5" H 14050 15155 50  0000 L CNN
-F 2 "MountingHole:MountingHole_2.7mm" H 13950 15200 50  0001 C CNN
+F 2 "MountingHole:MountingHole_2.2mm_M2" H 13950 15200 50  0001 C CNN
 F 3 "~" H 13950 15200 50  0001 C CNN
 F 4 "DNP" H 13950 15200 50  0001 C CNN "DNP"
@@
 F 0 "H6" H 14050 15446 50  0000 L CNN
 F 1 "M2.5" H 14050 15355 50  0000 L CNN
-F 2 "MountingHole:MountingHole_2.7mm" H 13950 15400 50  0001 C CNN
+F 2 "MountingHole:MountingHole_2.2mm_M2" H 13950 15400 50  0001 C CNN
 F 3 "~" H 13950 15400 50  0001 C CNN
 F 4 "DNP" H 13950 15400 50  0001 C CNN "DNP"
@@
 F 0 "H12" H 14650 15446 50  0000 L CNN
 F 1 "M2.5" H 14650 15355 50  0000 L CNN
-F 2 "MountingHole:MountingHole_2.7mm" H 14550 15400 50  0001 C CNN
+F 2 "MountingHole:MountingHole_2.2mm_M2" H 14550 15400 50  0001 C CNN
 F 3 "~" H 14550 15400 50  0001 C CNN
 F 4 "DNP" H 14550 15400 50  0001 C CNN "DNP"
@@
 F 0 "H11" H 14650 15246 50  0000 L CNN
 F 1 "M2.5" H 14650 15155 50  0000 L CNN
-F 2 "MountingHole:MountingHole_2.7mm" H 14550 15200 50  0001 C CNN
+F 2 "MountingHole:MountingHole_2.2mm_M2" H 14550 15200 50  0001 C CNN
 F 3 "~" H 14550 15200 50  0001 C CNN
 F 4 "DNP" H 14550 15200 50  0001 C CNN "DNP"
@@
 F 0 "H10" H 14650 15046 50  0000 L CNN
 F 1 "M2.5" H 14650 14955 50  0000 L CNN
-F 2 "MountingHole:MountingHole_2.7mm" H 14550 15000 50  0001 C CNN
+F 2 "MountingHole:MountingHole_2.2mm_M2" H 14550 15000 50  0001 C CNN
 F 3 "~" H 14550 15000 50  0001 C CNN
 F 4 "DNP" H 14550 15000 50  0001 C CNN "DNP"
@@
 F 0 "H9" H 14650 14846 50  0000 L CNN
 F 1 "M2.5" H 14650 14755 50  0000 L CNN
-F 2 "MountingHole:MountingHole_2.7mm" H 14550 14800 50  0001 C CNN
+F 2 "MountingHole:MountingHole_2.2mm_M2" H 14550 14800 50  0001 C CNN
 F 3 "~" H 14550 14800 50  0001 C CNN
 F 4 "DNP" H 14550 14800 50  0001 C CNN "DNP"
@@
 F 0 "H8" H 14650 14646 50  0000 L CNN
 F 1 "M2.5" H 14650 14555 50  0000 L CNN
-F 2 "MountingHole:MountingHole_2.7mm" H 14550 14600 50  0001 C CNN
+F 2 "MountingHole:MountingHole_2.2mm_M2" H 14550 14600 50  0001 C CNN
 F 3 "~" H 14550 14600 50  0001 C CNN
 F 4 "DNP" H 14550 14600 50  0001 C CNN "DNP"
@@
 F 0 "H7" H 14650 14446 50  0000 L CNN
 F 1 "M2.5" H 14650 14355 50  0000 L CNN
-F 2 "MountingHole:MountingHole_2.7mm" H 14550 14400 50  0001 C CNN
+F 2 "MountingHole:MountingHole_2.2mm_M2" H 14550 14400 50  0001 C CNN
 F 3 "~" H 14550 14400 50  0001 C CNN
 F 4 "DNP" H 14550 14400 50  0001 C CNN "DNP"
