File: hardware/lower-plate/keyboard.kicad_pcb (KiCad board)
At the start: 2 copper layers, 390 x 120.2 mm, 13 parts

Commit message: update mounting hole locations
Parts:
- moved H9 0.51 mm to (157.1, 109.5)
- moved H4 0.40 mm to (461.6, 128.5)
- moved H10 0.30 mm to (138.0, 185.7)
- moved H1 0.20 mm to (119.0, 166.7)

Commit message: mechanical changes
Parts:
- H1, H10, H11, H12, H2, H3, H4, H5, H6, H7, H8, H9: footprint MountingHole:MountingHole_2.7mm -> MountingHole:MountingHole_2.2mm_M2

Commit message: add encoder top right
Parts:
- LOGO4: moved to F.Cu
- moved LOGO4 0.11 mm to (290.1, 147.2), turned to 0 degrees
