File: hardware/0.3-w/keyboard.kicad_sch (KiCad schematic)
At the start: 272 parts, among them J1 USB_C_Receptacle_USB2.0, J2 SWD, J3 JST_PH2, Q1 AO3401A, Q2 2N7002, Q3 2N7002, SW1 RESET, U1 TP4057, U2 SRV05-4, U3 XC6206PxxxMR, U4 nRF52840_holyiot_18010

Commit message: clean up layout
Parts:
- D14: value PINK -> BLU
- D2: value BLU -> PNK
- U3: value XC6206PxxxMR -> XC6206P332MR
Changed lines of the file:
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@@
       (effects (font (size 1.27 1.27)) (justify right))
     )
-    (property "Value" "PINK" (id 1) (at 199.2122 248.9708 90)
+    (property "Value" "BLU" (id 1) (at 199.2122 248.9708 90)
       (effects (font (size 1.27 1.27)) (justify right))
     )
@@
       (effects (font (size 1.27 1.27)) (justify right))
     )
-    (property "Value" "BLU" (id 1) (at 310.2611 249.3783 90)
+    (property "Value" "PNK" (id 1) (at 310.2611 249.3783 90)
       (effects (font (size 1.27 1.27)) (justify right))
     )
@@
     (in_bom yes) (on_board yes)
     (property "Reference" "U3" (id 0) (at 271.78 263.9018 0))
-    (property "Value" "XC6206PxxxMR" (id 1) (at 278.13 266.2005 0))
+    (property "Value" "XC6206P332MR" (id 1) (at 278.13 266.2005 0))
     (property "Footprint" "Package_TO_SOT_SMD:SOT-23" (id 2) (at 275.59 263.525 0)
       (effects (font (size 1.27 1.27) italic) hide)
@@
     )
     (path "/58feb3e0-5b67-4960-9ce9-f4d263ded301"
-      (reference "D2") (unit 1) (value "BLU") (footprint "LED_SMD:LED_0603_1608Metric")
+      (reference "D2") (unit 1) (value "PNK") (footprint "LED_SMD:LED_0603_1608Metric")
     )
     (path "/00000000-0000-0000-0000-00005ef17407"
-      (reference "D14") (unit 1) (value "PINK") (footprint "LED_SMD:LED_0603_1608Metric")
+      (reference "D14") (unit 1) (value "BLU") (footprint "LED_SMD:LED_0603_1608Metric")
     )
     (path "/00000000-0000-0000-0000-0000691f43dd"
@@
     )
     (path "/cab1380b-6d0f-496d-8af6-dc3d54a48f02"
-      (reference "U3") (unit 1) (value "XC6206PxxxMR") (footprint "Package_TO_SOT_SMD:SOT-23")
+      (reference "U3") (unit 1) (value "XC6206P332MR") (footprint "Package_TO_SOT_SMD:SOT-23")
     )
     (path "/2502cfc3-64c2-41a8-8a9e-f1d40ca0e317"

Commit message: finalise 0.3w
Parts:
- C3: JLCSMT (none) -> C19702; LCSC (none) -> C19702; MPN (none) -> CL10A106KP8NNNC; Manufacturer (none) -> Samsung Electro-Mechanics
- C4: JLCSMT (none) -> C15849; LCSC (none) -> C15849; MPN (none) -> CL10A105KB8NNNC; Manufacturer (none) -> Samsung Electro-Mechanics
- D1: Manufacturer Hubei KENTO Elec -> Hubei KENTO Elec
- D14: JLCSMT C2286 -> C72041; LCSC C2286 -> C72041; MPN KT-0603R -> 19-217/BHC-ZL1M2RY/3T; Manufacturer Hubei KENTO Elec -> Everlight Elec
- D2: value PNK -> GRN; JLCSMT (none) -> C72043; LCSC (none) -> C72043; MPN (none) -> 19-217/GHC-YR1S2/3T; Manufacturer (none) -> Everlight Elec
- J1: JLCSMT (none) -> C165948; LCSC C319148 -> C165948; MPN U262-161N-4BVC11 -> TYPE-C-31-M-12; Manufacturer XKB Enterpriser -> Korean Hroparts Elec; Notes Sub: USB4105-GF-A (available at Digikey) -> (none)
- Q1: JLCSMT (none) -> C15127; LCSC (none) -> C15127; MPN (none) -> AO3401A; Manufacturer (none) -> Alpha & Omega Semicon
- Q2, Q3: JLCSMT (none) -> C8545; LCSC (none) -> C8545; MPN (none) -> 2N7002; Manufacturer (none) -> Changjiang Electronics Tech (CJ)
- R10, R9: JLCSMT (none) -> C25804; LCSC (none) -> C25804; MPN (none) -> 0603WAF1002T5E; Manufacturer (none) -> Uniroyal Elec
- R12: JLCSMT (none) -> C23186; LCSC (none) -> C23186; MPN (none) -> 0603WAF5101T5E; Manufacturer (none) -> Uniroyal Elec
- R7: JLCSMT (none) -> C23250; LCSC (none) -> C23250; MPN (none) -> 0603WAF8063T5E; Manufacturer (none) -> Uniroyal Elec
- R8: JLCSMT (none) -> C22976; LCSC (none) -> C22976; MPN (none) -> 0603WAF2004T5E; Manufacturer (none) -> Uniroyal Elec
- SW1: JLCSMT (none) -> C99271; LCSC (none) -> C99271; MPN (none) -> KMR231GLFS; Manufacturer (none) -> C&K
- U1: JLCSMT (none) -> C12044; LCSC (none) -> C12044; MPN (none) -> TP4057-42-SOT26-R; Manufacturer (none) -> TOPPOWER
- U2: JLCSMT (none) -> C85364; LCSC (none) -> C85364; MPN (none) -> SRV05-4-P-T7; Manufacturer (none) -> ProTek Devices
- U3: JLCSMT (none) -> C5446; LCSC (none) -> C5446; MPN (none) -> XC6206P332MR; Manufacturer (none) -> Torex Semicon
Other:
- note added: "Move Row3 down here"
