File: hardware/0.4-w/keyboard.kicad_sch (KiCad schematic)
At the start: 309 parts, among them J1 JST_PH2, J2 USB_C_Receptacle_USB2.0, J3 SWD, Q1 AO3401A, Q2 2N7002, Q3 AO3401A, SW1 RESET, U1 XC6206P332MR, U2 TP4057, U3 SRV05-4, U4 nRF52840_holyiot_18010, U5 SN74LVC1T45DBV

Commit message: clean up routing
Parts:
- removed C4: 10u, Capacitor_SMD:C_0603_1608Metric, symbol Device:C
- added C22: 10u, Capacitor_SMD:C_0603_1608Metric, symbol Device:C
- D21: renamed from D24; JLCSMT (none) -> C122853; LCSC (none) -> C122853; MPN (none) -> B5817WL; Manufacturer (none) -> Shikues
- R10: value 100K -> 806K; JLCSMT (none) -> C23250; LCSC (none) -> C23250; MPN (none) -> 0603WAF8063T5E; Manufacturer (none) -> Uniroyal Elec
- renumbered C15 to C1, C24 to C10, C10 to C11, C11 to C13, C22 to C15, C13 to C16, C16 to C17, C25 to C18, C6 to C19, C23 to C2, C7 to C20, C5 to C21, C28 to C23, C1 to C24, C2 to C25, C3 to C26, C20 to C27, C27 to C3, C17 to C4, C21 to C5, C8 to C6, C26 to C7, C29 to C8, D20 to D1, D5 to D10, D13 to D11, D4 to D12, D14 to D13, D3 to D14, D2 to D16, D16 to D17, D1 to D18, D18 to D19, D21 to D2, D17 to D20, D19 to D22, D9 to D23, D10 to D24, D22 to D3, D23 to D4, D8 to D5, D11 to D6, D6 to D8, D12 to D9, D_20 to D_1, D_94 to D_10, D_42 to D_100, D_61 to D_101, D_79 to D_102, D_1 to D_103, D_22 to D_104, D_41 to D_105, D_60 to D_106, D_97 to D_107, D_78 to D_108, D_2 to D_109, D_58 to D_11, D_21 to D_110, D_96 to D_111, D_76 to D_12, D_18 to D_13, D_109 to D_14, D_93 to D_15, D_57 to D_16, D_38 to D_17, D_17 to D_18, D_108 to D_19, D_40 to D_2, D_37 to D_20, D_75 to D_21, D_56 to D_22, D_92 to D_23, D_16 to D_24, D_36 to D_25, D_107 to D_26, D_74 to D_27, D_55 to D_28, D_91 to D_29, D_59 to D_3, D_106 to D_30, D_15 to D_31, D_35 to D_32, D_73 to D_33, D_54 to D_34, D_90 to D_35, D_14 to D_36, D_34 to D_37, D_72 to D_38, D_53 to D_39, D_77 to D_4, D_105 to D_40, D_89 to D_41, D_13 to D_42, D_33 to D_43, D_71 to D_44, D_52 to D_45, D_88 to D_46, D_12 to D_47, D_32 to D_48, D_70 to D_49, D_111 to D_5, D_104 to D_50, D_87 to D_52, D_11 to D_53, D_31 to D_54, D_69 to D_55, D_50 to D_56, D_86 to D_57, D_10 to D_58, D_30 to D_59, D_95 to D_6, D_68 to D_60, D_103 to D_61, D_49 to D_62, D_85 to D_63, D_9 to D_64, D_29 to D_65, D_67 to D_66, D_48 to D_67, D_84 to D_68, D_8 to D_69, D_39 to D_7, D_28 to D_70, D_66 to D_71, D_102 to D_72, D_47 to D_73, D_83 to D_74, D_7 to D_75, D_27 to D_76, D_65 to D_77, D_46 to D_78, D_101 to D_79, D_19 to D_8, D_6 to D_80, D_26 to D_81, D_64 to D_83, D_45 to D_84, D_100 to D_85, D_5 to D_86, D_25 to D_87, D_24 to D_88, D_99 to D_89, D_110 to D_9, D_81 to D_90, D_44 to D_91, D_63 to D_92, D_4 to D_93, D_43 to D_94, D_62 to D_95, D_23 to D_96, D_80 to D_97, D_3 to D_99, J3 to J1, J1 to J3, JP2 to JP1, JP1 to JP2, K_17 to K_1, K_23 to K_10, K_102 to K_100, K_58 to K_101, K_95 to K_102, K_14 to K_103, K_39 to K_104, K_116 to K_105, K_78 to K_106, K_40 to K_107, K_59 to K_108, K_15 to K_109, K_43 to K_11, K_21 to K_110, K_96 to K_111, K_117 to K_112, K_16 to K_113, K_41 to K_114, K_60 to K_115, K_79 to K_116, K_97 to K_117, K_63 to K_12, K_81 to K_13, K_104 to K_14, K_19 to K_15, K_24 to K_16, K_44 to K_17, K_64 to K_18, K_82 to K_19, K_22 to K_2, K_105 to K_20, K_106 to K_21, K_20 to K_22, K_25 to K_23, K_45 to K_24, K_65 to K_25, K_83 to K_26, K_99 to K_27, K_1 to K_28, K_26 to K_29, K_42 to K_3, K_107 to K_30, K_46 to K_31, K_66 to K_32, K_84 to K_33, K_2 to K_34, K_27 to K_35, K_108 to K_36, K_47 to K_37, K_67 to K_38, K_3 to K_39, K_62 to K_4, K_28 to K_40, K_85 to K_41, K_48 to K_42, K_109 to K_43, K_68 to K_44, K_4 to K_45, K_29 to K_46, K_86 to K_47, K_49 to K_48, K_69 to K_49, K_61 to K_5, K_5 to K_50, K_30 to K_51, K_87 to K_52, K_50 to K_53, K_110 to K_54, K_70 to K_55, K_6 to K_56, K_31 to K_57, K_88 to K_58, K_51 to K_59, K_80 to K_6, K_71 to K_60, K_7 to K_61, K_32 to K_62, K_89 to K_63, K_111 to K_64, K_52 to K_65, K_100 to K_66, K_72 to K_67, K_8 to K_68, K_33 to K_69, K_103 to K_7, K_90 to K_70, K_53 to K_71, K_73 to K_72, K_9 to K_73, K_34 to K_74, K_91 to K_75, K_112 to K_76, K_54 to K_77, K_74 to K_78, K_10 to K_79, K_98 to K_8, K_35 to K_80, K_92 to K_81, K_55 to K_82, K_75 to K_83, K_11 to K_84, K_36 to K_85, K_101 to K_86, K_93 to K_87, K_113 to K_88, K_56 to K_89, K_18 to K_9, K_76 to K_90, K_12 to K_91, K_37 to K_92, K_114 to K_93, K_57 to K_95, K_77 to K_96, K_115 to K_97, K_13 to K_98, K_38 to K_99, LOGO2 to LOGO1, LOGO1 to LOGO2, Q2 to Q1, Q1 to Q2, R2 to R1, R7 to R2, R4 to R3, R3 to R4, R8 to R5, R1 to R6, R5 to R7, R6 to R8, U4 to U1, U5 to U2, U1 to U3, U3 to U4, U2 to U5
Connections:
- net GND: now also C22.2
- net at D21.1 (K), Q3.2 (S), U3.3 (VI): now also C22.1

Commit message: 0.4 cleanup and 0.5 addition of files
Parts:
- added J4: Spare IO, josh-connectors:4_PIN_THT_Staggered, symbol Connector:Conn_01x04_Male
- added K_120: KEYSW, josh-keyboard:MXOnly-1.5U-NoLED, symbol josh-keyboard:MX-NoLED
- added K_121: KEYSW, josh-keyboard:MXOnly-1U-NoLED, symbol josh-keyboard:MX-NoLED
- R11: value 1K -> 2K; JLCSMT C21190 -> (none); LCSC C21190 -> (none); MPN 0603WAF1001T5E -> (none); Manufacturer Uniroyal Elec -> (none)
- R8: value 5K1 -> 2K; JLCSMT C23186 -> (none); LCSC C23186 -> (none); MPN 0603WAF5101T5E -> (none); Manufacturer Uniroyal Elec -> (none)
- U2: footprint Package_TO_SOT_SMD:SOT-23-6 -> Package_TO_SOT_SMD:SOT-363_SC-70-6
Connections:
- net COL4: now also K_120.1 (COL)
- net COL5: now also K_121.1 (COL)
- net GND: now also J4.4 (Pin_4)
- net at D_85.2 (A), K_30.2 (ROW): now also K_120.2 (ROW)
- net at D_79.2 (A), K_36.2 (ROW): now also K_121.2 (ROW)
- net SPARE_2: now reaches U1.42 (P1.08)
- net SPARE_2: now also J4.3 (Pin_3)
- net SPARE_0: now reaches U1.54 (P0.13)
- net SPARE_0: now also J4.1 (Pin_1)
- net SPARE_1: now reaches U1.55 (P0.16)
- net SPARE_1: now also J4.2 (Pin_2)
- no-connect marks 10 -> 7
Other:
- note added: "2K = 400mA Charge"
- note added: "Spare"
- note removed: "5K1 = 200mA Charge"
- moved on the sheet: K_30, K_36, K_43
